File: pcb/funkyboi.kicad_sch (KiCad schematic)
At the start: 70 parts, among them J1 Conn_01x10, J10 Conn_01x01, J11 Conn_01x01, J12 Conn_01x02, J13 Conn_01x02, J14 Conn_01x02, J15 Conn_01x01, J16 Conn_01x01, J17 Conn_01x01, J18 Conn_01x02, J19 Conn_01x01, J20 Conn_01x01, J3 Conn_01x05, J4 Conn_01x10, J5 Conn_Pi_SWD, J6 Conn_Pi_UART, J7 LCD_ST7789, J8 I2S_AUDIO, J9 Conn_01x02, Q1 BSS84, SW1 SW_RESET, SW10 START, SW2 SW_BOOTSEL, SW3 UP, SW4 LEFT, SW5 RIGHT, SW6 DOWN, SW7 B, SW8 A, SW9 SELECT, U1 W25Q128JVPIQ, U2 ME4055, U3 ME6211, U4 FLASH or PSRAM, U5 RP2350B, Y1 CM4012M00012001

Commit message: revision 1 update
Parts:
- removed J1, J4: Conn_01x10, Connector_PinHeader_1.27mm:PinHeader_1x10_P1.27mm_Vertical, symbol Connector_Generic:Conn_01x10
- removed J10, J11, J15, J16, J17, J19, J20: Conn_01x01, Connector_PinHeader_1.27mm:PinHeader_1x01_P1.27mm_Vertical, symbol Connector_Generic:Conn_01x01
- removed J12, J13, J14, J18, J9: Conn_01x02, Connector_PinHeader_1.27mm:PinHeader_1x02_P1.27mm_Vertical, symbol Connector_Generic:Conn_01x02
- removed J3: Conn_01x05, Connector_PinHeader_1.27mm:PinHeader_1x05_P1.27mm_Vertical, symbol Connector_Generic:Conn_01x05
- removed J7: LCD_ST7789, Connector_PinHeader_2.54mm:PinHeader_1x08_P2.54mm_Vertical, symbol Connector_Generic:Conn_01x08
- removed J8: I2S_AUDIO, Connector_PinHeader_2.54mm:PinHeader_1x05_P2.54mm_Vertical, symbol Connector_Generic:Conn_01x05
- removed SW10: START, Button_Switch_SMD:SW_SPST_B3U-1000P, symbol Switch:SW_SPST
- removed SW3: UP, Button_Switch_SMD:SW_SPST_B3U-1000P, symbol Switch:SW_SPST
- removed SW4: LEFT, Button_Switch_SMD:SW_SPST_B3U-1000P, symbol Switch:SW_SPST
- removed SW5: RIGHT, Button_Switch_SMD:SW_SPST_B3U-1000P, symbol Switch:SW_SPST
- removed SW6: DOWN, Button_Switch_SMD:SW_SPST_B3U-1000P, symbol Switch:SW_SPST
- removed SW7: B, Button_Switch_SMD:SW_SPST_B3U-1000P, symbol Switch:SW_SPST
- removed SW8: A, Button_Switch_SMD:SW_SPST_B3U-1000P, symbol Switch:SW_SPST
- removed SW9: SELECT, Button_Switch_SMD:SW_SPST_B3U-1000P, symbol Switch:SW_SPST
- added J1: BUTTONS, Connector_PinHeader_1.27mm:PinHeader_1x08_P1.27mm_Vertical, symbol Connector_Generic:Conn_01x08
- added J10, J8: Conn_01x07, Connector_PinHeader_1.27mm:PinHeader_1x07_P1.27mm_Vertical, symbol Connector_Generic:Conn_01x07
- added J2: ST7789, Connector_PinSocket_2.54mm:PinSocket_1x07_P2.54mm_Vertical, symbol Connector_Generic:Conn_01x07
- added J4: Conn_01x06, Connector_PinHeader_1.27mm:PinHeader_1x06_P1.27mm_Vertical, symbol Connector_Generic:Conn_01x06
- added J7: MAX98357, Connector_PinHeader_2.54mm:PinHeader_1x07_P2.54mm_Vertical, symbol Connector_Generic:Conn_01x07
- added J9: Conn_01x18, Connector_PinHeader_1.27mm:PinHeader_1x18_P1.27mm_Vertical, symbol Connector_Generic:Conn_01x18
Connections:
- net +3V3: now also J2.2 (Pin_2), J7.7 (Pin_7)
- net +5V: now also J9.12 (Pin_12)
- net BAT_STAT: now also J9.9 (Pin_9)
- net BOOTSEL: now also J9.17 (Pin_17)
- net GND: now also J2.1 (Pin_1), J7.6 (Pin_6)
- net GPIO10: now also J10.4 (Pin_4)
- net GPIO11: now also J10.5 (Pin_5)
- net GPIO12: now also J10.6 (Pin_6)
- net GPIO13: now also J10.7 (Pin_7)
- net GPIO14: now also J7.1 (Pin_1)
- net GPIO18: now also J7.5 (Pin_5)
- net GPIO19: now also J4.1 (Pin_1)
- net GPIO2: now also J2.3 (Pin_3)
- net GPIO20: now also J4.2 (Pin_2)
- net GPIO21: now also J4.3 (Pin_3)
- net GPIO22: now also J4.4 (Pin_4)
- net GPIO23: now also J4.5 (Pin_5)
- net GPIO24: now also J4.6 (Pin_6)
- net GPIO25: now also J1.1 (Pin_1)
- net GPIO26: now also J1.2 (Pin_2)
- net GPIO27: now also J1.3 (Pin_3)
- net GPIO28: now also J1.4 (Pin_4)
- net GPIO29: now also J1.5 (Pin_5)
- net GPIO3: now also J2.4 (Pin_4)
- net GPIO30: now also J1.6 (Pin_6)
- net GPIO31: now also J1.7 (Pin_7)
- net GPIO32: now also J1.8 (Pin_8)
- net GPIO33: now also J8.1 (Pin_1)
- net GPIO34: now also J8.2 (Pin_2)
- net GPIO35: now also J8.3 (Pin_3)
- net GPIO36: now also J8.4 (Pin_4)
- net GPIO37: now also J8.5 (Pin_5)
- net GPIO38: now also J8.6 (Pin_6)
- net GPIO39: now also J8.7 (Pin_7)
- net GPIO4: now also J2.5 (Pin_5)
- net GPIO40: now also J9.1 (Pin_1)
- net GPIO41: now also J9.2 (Pin_2)
- net GPIO42: now also J9.3 (Pin_3)
- net GPIO43: now also J9.4 (Pin_4)
- net GPIO44: now also J9.5 (Pin_5)
- net GPIO45: now also J9.6 (Pin_6)
- net GPIO46: now also J9.7 (Pin_7)
- net GPIO47: now also J9.8 (Pin_8)
- net GPIO7: now also J10.1 (Pin_1)
- net GPIO8: now also J10.2 (Pin_2)
- net GPIO9: now also J10.3 (Pin_3)
- net LDO_EN: now also J9.10 (Pin_10)
- net SWCLK: now also J9.16 (Pin_16)
- net SWDIO: now also J9.15 (Pin_15)
- net USB_D+: now also J9.14 (Pin_14)
- net USB_D-: now also J9.13 (Pin_13)
- net VBAT: now also J9.11 (Pin_11)
- net ~{RESET}: now also J9.18 (Pin_18)
- net GPIO15 renamed BCLK
- net BCLK: now also J7.2 (Pin_2)
- net GPIO16 renamed DIN
- net DIN: now also J7.3 (Pin_3)
- net GPIO17 renamed GAIN
- net GAIN: now also J7.4 (Pin_4)
- net GPIO5 renamed DC
- net DC: now also J2.6 (Pin_6)
- net GPIO6 renamed BLK
- net BLK: now also J2.7 (Pin_7)
Other:
- note removed: "HANDHELD I/O Buttons: GPIO0/1/2/3, GPIO35/37, GPIO18/24 LCD: GPIO40-45 I2S audio: GPIO14-16"
